File: p02r00b01_14-10-28/BLEmodule.sch (KiCad schematic (older format))
At the start: 31 parts, among them IC1 NRF51822, P1 AIN_0_3, P2 CONN_2, P3 AIN_4_7, SW1 SWITCH-4, SW2 SWITCH-4, U1 ANTENNA-NC, X1 NX2520SA

Commit message: adding more files. Still dont know what am i doing.
Parts:
- removed B1: BALUN-JOHANSON, symbol BALUN-JOHANSON
- removed BT1: BATTERY, symbol BATTERY
- removed C1: 1uF, symbol C
- removed C10: 47nF, symbol C
- removed C11, C8: 0.1uF, symbol C
- removed C12: 2.2nF, symbol C
- removed C2: 10uF, symbol C
- removed C3: 4.7uF, symbol C
- removed C4, C7: 100nF, symbol C
- removed C5, C6: 12pF, ~, symbol C
- removed C9: 1nF, symbol C
- removed D1: DIODE, symbol DIODE
- removed D2, D3: LED, symbol LED
- removed IC1: NRF51822, symbol NRF51822
- removed L1: 15nH, symbol INDUCTOR
- removed L2: INDUCTOR, symbol INDUCTOR
- removed L3: 10uH, symbol INDUCTOR
- removed P1: AIN_0_3, symbol CONN_6
- removed P2: CONN_2, ~, symbol CONN_2
- removed P3: AIN_4_7, symbol CONN_6
- removed R1, R2: 100R, symbol R
- removed R3: 12K, symbol R
- removed SW1, SW2: SWITCH-4, symbol SWITCH-4
- removed U1: ANTENNA-NC, symbol ANTENNA-NC
- removed X1: NX2520SA, symbol CONN_4
- added B?: BALUN-JOHANSON, symbol BALUN-JOHANSON
- added BT?: BATTERY, symbol BATTERY
- added C?: 1uF, symbol C
- added C?: 4.7uF, symbol C
- added C? (x2): 100nF, symbol C
- added C?: 1nF, symbol C
- added C?: 2.2nF, symbol C
- added C?: 47nF, symbol C
- added C?: 10uF, symbol C
- added C? (x2): 0.1uF, symbol C
- added C? (x2): 12pF, ~, symbol C
- added D? (x2): LED, symbol LED
- added D?: DIODE, symbol DIODE
- added IC?: NRF51822, symbol NRF51822
- added L?: 10uH, symbol INDUCTOR
- added L?: 15nH, symbol INDUCTOR
- added L?: INDUCTOR, symbol INDUCTOR
- added P?: AIN_0_3, symbol CONN_6
- added P?: AIN_4_7, symbol CONN_6
- added P?: CONN_2, ~, symbol CONN_2
- added R?: 12K, symbol R
- added R? (x2): 100R, symbol R
- added SW? (x2): SWITCH-4, symbol SWITCH-4
- added U?: ANTENNA-NC, symbol ANTENNA-NC
- added X?: NX2520SA, symbol CONN_4
